Commit message: Fixed the Robot diffrential drive problem + changed the screenshot + removed my_plugin

File: my_robot/urdf/my_robot.xacro (robot description, xacro)
@@ -22,5 +22,5 @@
       <origin xyz="0 0 0" rpy=" 0 0 0"/>
       <geometry>
-        <box size=".8 .2 .1"/>
+        <box size=".8 .5 .1"/>
       </geometry>
     </collision>
@@ -28,5 +28,5 @@
       <origin xyz="0 0 0" rpy=" 0 0 0"/>
       <geometry>
-        <box size=".8 .2 .1"/>
+        <box size=".8 .5 .1"/>
       </geometry>
       <material name="chassis_material">
@@ -35,29 +35,4 @@
     </visual>
   </link>
-  <link name="left_wheel">
-  <pose>0 0 0 0 0 0</pose>
-  <!-- -0.15 -0.2 0.1 -->
-  <visual>
-    <origin xyz="0 0 0" rpy="0 1.5707 1.5707"/>
-   <geometry>
-    <cylinder radius="0.1" length="0.05"/>
-   </geometry>
-  </visual>
-  <collision>
-    <origin xyz="0 0 0" rpy="0 1.5707 1.5707"/>
-   <geometry>
-    <cylinder radius="0.1" length="0.05"/>
-   </geometry>
-  </collision>
-  <inertial>
-      <mass value="5.0"/>
-      <origin xyz="0.0 0 0" rpy=" 0 0 0"/>
-      <inertia
-          ixx="0.1" ixy="0" ixz="0"
-          iyy="0.1" iyz="0"
-          izz="0.1"
-      />
-    </inertial>
-  </link>
    <link name="left_front_wheel">
   <pose>0 0 0 0 0 0</pose>
@@ -110,29 +85,4 @@
     </inertial>
   </link>
-<link name="right_wheel">
-  <pose>0 0 0 0 0 0</pose>
-  <!-- -0.15 -0.2 0.1 -->
-  <visual>
-    <origin xyz="0 0 0" rpy="0 1.5707 1.5707"/>
-   <geometry>
-    <cylinder radius="0.1" length="0.05"/>
-   </geometry>
-  </visual>
-  <collision>
-    <origin xyz="0 0 0" rpy="0 1.5707 1.5707"/>
-   <geometry>
-    <cylinder radius="0.1" length="0.05"/>
-   </geometry>
-  </collision>
-  <inertial>
-      <mass value="5.0"/>
-      <origin xyz="0.0 0 0" rpy=" 0 0 0"/>
-      <inertia
-          ixx="0.1" ixy="0" ixz="0"
-          iyy="0.1" iyz="0"
-          izz="0.1"
-      />
-    </inertial>
-  </link>
 <link name="right_front_wheel">
   <pose>0 0 0 0 0 0</pose>
@@ -185,14 +135,6 @@
     </inertial>
   </link>
-  <joint type="continuous" name="left_wheel_hinge">
-    <origin xyz="0 0.15 0" rpy="0 0 0"/>
-    <child link="left_wheel"/>
-    <parent link="chassis"/>
-    <axis xyz="0 1 0" rpy="0 0 0"/>
-    <limit effort="10000" velocity="1000"/>
-    <dynamics damping="1.0" friction="1.0"/>
-  </joint>
   <joint type="continuous" name="left_front_wheel_hinge">
-    <origin xyz="0.3 0.15 0" rpy="0 0 0"/>
+    <origin xyz="0.3 0.3 0" rpy="0 0 0"/>
     <child link="left_front_wheel"/>
     <parent link="chassis"/>
@@ -202,5 +144,5 @@
   </joint>
   <joint type="continuous" name="left_back_wheel_hinge">
-    <origin xyz="-0.3 0.15 0" rpy="0 0 0"/>
+    <origin xyz="-0.3 0.3 0" rpy="0 0 0"/>
     <child link="left_back_wheel"/>
     <parent link="chassis"/>
@@ -210,5 +152,5 @@
   </joint>
   <joint type="continuous" name="right_front_wheel_hinge">
-    <origin xyz="0.3 -0.15 0" rpy="0 0 0"/>
+    <origin xyz="0.3 -0.3 0" rpy="0 0 0"/>
     <child link="right_front_wheel"/>
     <parent link="chassis"/>
@@ -218,14 +160,6 @@
   </joint>
    <joint type="continuous" name="right_back_wheel_hinge">
-    <origin xyz="-0.3 -0.15 0" rpy="0 0 0"/>
+    <origin xyz="-0.3 -0.3 0" rpy="0 0 0"/>
     <child link="right_back_wheel"/>
-    <parent link="chassis"/>
-    <axis xyz="0 1 0" rpy="0 0 0"/>
-    <limit effort="10000" velocity="1000"/>
-    <dynamics damping="1.0" friction="1.0"/>
-  </joint>
-   <joint type="continuous" name="right_wheel_hinge">
-    <origin xyz="0 -0.15 0" rpy="0 0 0"/>
-    <child link="right_wheel"/>
     <parent link="chassis"/>
     <axis xyz="0 1 0" rpy="0 0 0"/>
@@ -280,14 +214,8 @@
   <axis xyz="0 1 0"/>
 </joint>
-<gazebo reference="left_wheel">
-    <material>Gazebo/Brown</material>
-</gazebo>
 <gazebo reference="left_front_wheel">
     <material>Gazebo/Brown</material>
 </gazebo>
 <gazebo reference="left_back_wheel">
-    <material>Gazebo/Brown</material>
-</gazebo>
-<gazebo reference="right_wheel">
     <material>Gazebo/Brown</material>
 </gazebo>

Commit message: Fixed mentor robot sink feedback
Submitting the project

Uploaded the mapping database to google drive

File: my_robot/urdf/my_robot.xacro (robot description, xacro)
@@ -4,5 +4,5 @@
   <link name="robot_footprint"></link>
   <joint name="robot_footprint_joint" type="fixed">
-    <origin xyz="0 0 0" rpy="0 0 0" />
+    <origin xyz="0 0 0.1" rpy="0 0 0" />
     <parent link="robot_footprint"/>
     <child link="chassis" />
@@ -22,5 +22,5 @@
       <origin xyz="0 0 0" rpy=" 0 0 0"/>
       <geometry>
-        <box size=".8 .5 .1"/>
+        <box size=".42 .5 .1"/>
       </geometry>
     </collision>
@@ -28,5 +28,5 @@
       <origin xyz="0 0 0" rpy=" 0 0 0"/>
       <geometry>
-        <box size=".8 .5 .1"/>
+        <box size=".42 .5 .1"/>
       </geometry>
       <material name="chassis_material">
@@ -136,5 +136,5 @@
   </link>
   <joint type="continuous" name="left_front_wheel_hinge">
-    <origin xyz="0.3 0.3 0" rpy="0 0 0"/>
+    <origin xyz="0.11 0.3 0" rpy="0 0 0"/>
     <child link="left_front_wheel"/>
     <parent link="chassis"/>
@@ -144,5 +144,5 @@
   </joint>
   <joint type="continuous" name="left_back_wheel_hinge">
-    <origin xyz="-0.3 0.3 0" rpy="0 0 0"/>
+    <origin xyz="-0.11 0.3 0" rpy="0 0 0"/>
     <child link="left_back_wheel"/>
     <parent link="chassis"/>
@@ -152,5 +152,5 @@
   </joint>
   <joint type="continuous" name="right_front_wheel_hinge">
-    <origin xyz="0.3 -0.3 0" rpy="0 0 0"/>
+    <origin xyz="0.11 -0.3 0" rpy="0 0 0"/>
     <child link="right_front_wheel"/>
     <parent link="chassis"/>
@@ -160,5 +160,5 @@
   </joint>
    <joint type="continuous" name="right_back_wheel_hinge">
-    <origin xyz="-0.3 -0.3 0" rpy="0 0 0"/>
+    <origin xyz="-0.11 -0.3 0" rpy="0 0 0"/>
     <child link="right_back_wheel"/>
     <parent link="chassis"/>
@@ -167,5 +167,5 @@
     <dynamics damping="1.0" friction="1.0"/>
   </joint>
-<link name="camera">
+<link name="camera_link">
   <origin xyz="0 0 0" rpy="0 0 0"/>
   <visual>
@@ -186,7 +186,7 @@
 </link>
 <joint name="camera_joint" type="fixed">
-  <origin xyz="0.4 0 0" rpy="0 0 0"/>
+  <origin xyz="0.21 0 0" rpy="0 0 0"/>
   <parent link="chassis"/>
-  <child link="camera"/>
+  <child link="camera_link"/>
   <axis xyz="0 1 0"/>
 </joint>
@@ -209,5 +209,5 @@
 </link>
 <joint name="hokuyo_joint" type="fixed">
-  <origin xyz="0.4 0 0.1" rpy="0 0 0"/>
+  <origin xyz="0.21 0 0.1" rpy="0 0 0"/>
   <parent link="chassis"/>
   <child link="hokuyo"/>
@@ -215,20 +215,27 @@
 </joint>
 <gazebo reference="left_front_wheel">
-    <material>Gazebo/Brown</material>
+    <material>Gazebo/Blue</material>
 </gazebo>
 <gazebo reference="left_back_wheel">
-    <material>Gazebo/Brown</material>
+    <material>Gazebo/Blue</material>
 </gazebo>
 <gazebo reference="right_front_wheel">
-    <material>Gazebo/Brown</material>
+    <material>Gazebo/Blue</material>
 </gazebo>
 <gazebo reference="right_back_wheel">
-    <material>Gazebo/Brown</material>
+    <material>Gazebo/Blue</material>
 </gazebo>
 <gazebo reference="chassis">
     <material>Gazebo/Green</material>
 </gazebo>
-<gazebo reference="camera">
+<gazebo reference="camera_link">
     <material>Gazebo/Red</material>
 </gazebo>
+<joint name="camera_optical_joint" type="fixed">
+    <origin xyz="0 0 0" rpy="-1.5707 0 -1.5707"/>
+    <parent link="camera_link"/>
+    <child link="camera_link_optical"/>
+</joint>
+<link name="camera_link_optical">
+</link>
 </robot>
